File: KiCAD/audio-addon-board-pcm1802/audio-addon-board-pcm1802.kicad_sch (KiCad schematic)
At the start: 63 parts, among them J1 RCA, J2 CONN_HOST_1, J3 RCA, J4 RCA, J5 RCA, SW1 SW_DIP_x04, U1 PCM1802DBR, U2 LTC1682IS8-5

Commit message: update board
Parts:
- D1: footprint LED_SMD:LED_0805_2012Metric -> LED_SMD:LED_0603_1608Metric
Changed lines of the file:
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@@
 			)
 		)
-		(property "Footprint" "LED_SMD:LED_0805_2012Metric"
+		(property "Footprint" "LED_SMD:LED_0603_1608Metric"
 			(at 168.91 62.23 0)
 			(effects
